Commit message: fix camera orientation and add depth camera

File: kinova_description/urdf/camera.xacro (robot description, xacro)
@@ -2,7 +2,7 @@
 <robot xmlns:xacro="http://www.ros.org/wiki/xacro" >
     <joint name="camera_joint" type="fixed">
-        <parent link="j2n6s300_link_6"/>
+        <parent link="j2n6s300_end_effector"/>
         <child link="camera_link"/>
-        <origin xyz="1 0 0" rpy="0 0 0"/>
+        <origin xyz="0 0 0" rpy="${pi/} ${-pi/2} 0"/>
     </joint>
     <link name="camera_link">
@@ -24,5 +24,5 @@
     <gazebo reference="camera_link">
         <material>Gazebo/Red</material>
-        <sensor name="camera" type="camera">
+        <sensor name="camera" type="depth">
             <pose> 0 0 0 0 0 0 </pose>
             <visualize>true</visualize>
@@ -42,4 +42,6 @@
             <plugin name="camera_controller" filename="libgazebo_ros_camera.so">
                 <frame_name>camera_link_optical</frame_name>
+                <min_depth>0.01</min_depth>
+                <max_depth>100.0</max_depth>
             </plugin>
         </sensor>

Commit message: fix camera position

File: kinova_description/urdf/camera.xacro (robot description, xacro)
@@ -4,5 +4,5 @@
         <parent link="j2n6s300_end_effector"/>
         <child link="camera_link"/>
-        <origin xyz="0 0 0" rpy="${pi/} ${-pi/2} 0"/>
+        <origin xyz="0 0 0" rpy="${pi} ${-pi/2} 0"/>
     </joint>
     <link name="camera_link">

Commit message: changed camera, rviz config for visualization

File: kinova_description/urdf/camera.xacro (robot description, xacro)
@@ -21,5 +21,11 @@
         <origin xyz="0 0 0" rpy="0 0 0"/>
     </joint>
+    <joint name="camera_coordinate_joint" type="fixed">
+        <parent link="camera_link"/>
+        <child link="camera_coordinate_system"/>
+        <origin xyz="0 0 0" rpy="${-pi/2} 0 ${-pi/2}"/>
+    </joint>
     <link name="camera_link_optical"></link>
+    <link name="camera_coordinate_system"></link>
     <gazebo reference="camera_link">
         <material>Gazebo/Red</material>
@@ -48,12 +54,13 @@
     <sensor name="world" type="depth">
         <!-- openni plugin has the x pointing towards the scene, so rotate to have z -->
-        <!--pose>0.0 0.0 1.0 0.0 -1.5708 1.5708</pose -->
-        <pose> 0 0 0 0 0 0 </pose>
+        <pose>0.0 0.0 1.0 0.0 -1.5708 1.5708</pose>
+        <!-- <pose> 0 0 0 0 0 0 </pose> -->
         <camera>
             <horizontal_fov>0.74839718</horizontal_fov>
             <image>
-                <width>1280</width>
-                <height>1024</height>
-                <format>L_INT8</format>
+                <width>640</width>
+                <height>480</height>
+                <format>R8G8B8</format>
+                <!-- <format>L_INT8</format> -->
             </image>
             <clip>
@@ -79,5 +86,5 @@
             <depthImageInfoTopicName>/3d_image/camera_info</depthImageInfoTopicName>
             <pointCloudTopicName>/3d_image/3d_cloud</pointCloudTopicName>
-            <frameName>camera_link_optical</frameName>
+            <frameName>camera_coordinate_system</frameName>
             <pointCloudCutoff>0.5</pointCloudCutoff>
             <pointCloudCutoffMax>2.0</pointCloudCutoffMax>

Commit message: added collision box

File: kinova_description/urdf/camera.xacro (robot description, xacro)
@@ -15,4 +15,9 @@
             </material>
         </visual>
+        <collision>
+            <geometry>
+                <box size="0.010 0.03 0.03"/>
+            </geometry>
+        </collision>
     </link>
     <joint name="camera_optical_joint" type="fixed">

Commit message: reduced collision box size

File: kinova_description/urdf/camera.xacro (robot description, xacro)
@@ -17,5 +17,5 @@
         <collision>
             <geometry>
-                <box size="0.010 0.03 0.03"/>
+                <box size="0.005 0.01 0.01"/>
             </geometry>
         </collision>

Commit message: removed collision box

File: kinova_description/urdf/camera.xacro (robot description, xacro)
@@ -15,9 +15,4 @@
             </material>
         </visual>
-        <collision>
-            <geometry>
-                <box size="0.005 0.01 0.01"/>
-            </geometry>
-        </collision>
     </link>
     <joint name="camera_optical_joint" type="fixed">

Commit message: add surgery room with blue floor

File: kinova_description/urdf/camera.xacro (robot description, xacro)
@@ -52,5 +52,5 @@
             </plugin>
         </sensor> -->
-    <sensor name="world" type="depth">
+    <sensor name="root" type="depth">
         <!-- openni plugin has the x pointing towards the scene, so rotate to have z -->
         <pose>0.0 0.0 1.0 0.0 -1.5708 1.5708</pose>

File: kinova_description/urdf/j2n6s300_standalone.xacro (robot description, xacro)
@@ -21,5 +21,5 @@
     <child link="root" />
     <parent link="world" />
-    <origin xyz="0 0 0" rpy="0 0 0" />
+    <origin xyz="2 1 0" rpy="0 0 0" />
   </joint>
   <xacro:property name="robot_root" value="root" />

Commit message: move camera position in front of fingers

File: kinova_description/urdf/camera.xacro (robot description, xacro)
@@ -4,5 +4,5 @@
         <parent link="j2n6s300_end_effector"/>
         <child link="camera_link"/>
-        <origin xyz="0 0 0" rpy="${pi} ${-pi/2} 0"/>
+        <origin xyz="0 0 0.15" rpy="${pi} ${-pi/2} 0"/>
     </joint>
     <link name="camera_link">

Commit message: different initial robot position, works sometimes

File: kinova_description/urdf/camera.xacro (robot description, xacro)
@@ -4,5 +4,5 @@
         <parent link="j2n6s300_end_effector"/>
         <child link="camera_link"/>
-        <origin xyz="0 0 0.15" rpy="${pi} ${-pi/2} 0"/>
+        <origin xyz="0 0 0.075" rpy="${pi} ${-pi/2} 0"/>
     </joint>
     <link name="camera_link">

Commit message: change camera position and color

File: kinova_description/urdf/camera.xacro (robot description, xacro)
@@ -4,5 +4,5 @@
         <parent link="j2n6s300_end_effector"/>
         <child link="camera_link"/>
-        <origin xyz="0 0 0.075" rpy="${pi} ${-pi/2} 0"/>
+        <origin xyz="0 0 0.055" rpy="${pi} ${-pi/2} 0"/>
     </joint>
     <link name="camera_link">
@@ -11,6 +11,6 @@
                 <box size="0.010 0.03 0.03"/>
             </geometry>
-            <material name="red">
-                <color rgba= "1 0 0 1"/>
+            <material name="black">
+                <color rgba= "0 0 0 1"/>
             </material>
         </visual>
@@ -29,5 +29,5 @@
     <link name="camera_coordinate_system"></link>
     <gazebo reference="camera_link">
-        <material>Gazebo/Red</material>
+        <material>Gazebo/Black</material>
         <!-- <sensor name="camera" type="depth">
             <pose> 0 0 0 0 0 0 </pose>
